Commit message: change racer mass

File: gym_pybullet_drones/assets/racer.urdf (robot description, URDF)
Before this commit: robot cf2, 6 links, 5 joints
Links:
- link base_link: mass 0.027 -> 0.81

Commit message: update floss values

File: gym_pybullet_drones/assets/racer.urdf (robot description, URDF)
Before this commit: robot cf2, 6 links, 5 joints
Links:
- link base_link: mass 0.81 -> 0.830

Commit message: Change km

File: gym_pybullet_drones/assets/racer.urdf (robot description, URDF)
Before this commit: robot cf2, 6 links, 5 joints
Links:
- link base_link: geometry collision cylinder length=.025 radius=.06; visual mesh filename=./cf2.dae scale=3 3 3
